File: 4digitSSD-MAX7219/4digitSSD-MAX7219CNG.sch (EAGLE design)
At the start: 5 parts, among them IC1 MAX7219CNG

Commit message: REV 20170118A
slight routing changes. Added power supply filter capacitor.
Parts:
- added C1: .1uF, rcl:C-USC1206
- CN1: value (none) -> Aux PWR
- CON1: value (none) -> uC CONN
Connections:
- removed net D5: IC1.DIG4
- removed net D6: IC1.DIG5
- removed net D7: IC1.DIG6
- removed net D8: IC1.DIG7
- removed net DOUT: IC1.DOUT
- net GND: now also C1.2
- net VCC: now also C1.1
Other:
- note removed: "Alternate Power Source"
Changed lines of the file:
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@@
 <part name="VR1" library="SparkFun-Resistors" deviceset="TRIMPOT" device="-PTH-10MM-KNOB-1/2W-10%" value="10k"/>
 <part name="GND2" library="supply1" deviceset="GND" device=""/>
-<part name="CN1" library="adafruit" deviceset="JST_2PIN" device="-THM"/>
-<part name="CON1" library="con-harting" deviceset="CON06" device=""/>
+<part name="CN1" library="adafruit" deviceset="JST_2PIN" device="-THM" value="Aux PWR"/>
+<part name="CON1" library="con-harting" deviceset="CON06" device="" value="uC CONN"/>
+<part name="C1" library="rcl" deviceset="C-US" device="C1206" value=".1uF"/>
 </parts>
 <sheets>
@@
 <text x="65.786" y="59.69" size="1.016" layer="117" ratio="0">SSD starts at Digit 1
 MAX721x starts at Digit 0</text>
-<text x="-15.24" y="33.02" size="1.016" layer="117" ratio="0">Alternate Power Source</text>
 </plain>
 <instances>
@@
 <instance part="U$1" gate="G$1" x="0" y="78.74"/>
 <instance part="VR1" gate="R?" x="33.02" y="33.02" rot="R90"/>
-<instance part="GND2" gate="1" x="38.1" y="27.94"/>
+<instance part="GND2" gate="1" x="40.64" y="30.48"/>
 <instance part="CN1" gate="G$1" x="7.62" y="25.4" rot="R270"/>
 <instance part="CON1" gate="G$1" x="63.5" y="81.28" rot="R180"/>
+<instance part="C1" gate="G$1" x="-7.62" y="30.48"/>
 </instances>
 <busses>
@@
 </segment>
 </net>
-<net name="D5" class="0">
-<segment>
-<pinref part="IC1" gate="G$1" pin="DIG4"/>
-<wire x1="73.66" y1="45.72" x2="81.28" y2="45.72" width="0.1524" layer="91"/>
-<label x="81.28" y="45.72" size="1.016" layer="95" ratio="0" xref="yes"/>
-</segment>
-</net>
-<net name="D7" class="0">
-<segment>
-<pinref part="IC1" gate="G$1" pin="DIG6"/>
-<wire x1="73.66" y1="40.64" x2="81.28" y2="40.64" width="0.1524" layer="91"/>
-<label x="81.28" y="40.64" size="1.016" layer="95" ratio="0" xref="yes"/>
-</segment>
-</net>
-<net name="D8" class="0">
-<segment>
-<pinref part="IC1" gate="G$1" pin="DIG7"/>
-<wire x1="73.66" y1="38.1" x2="81.28" y2="38.1" width="0.1524" layer="91"/>
-<label x="81.28" y="38.1" size="1.016" layer="95" ratio="0" xref="yes"/>
-</segment>
-</net>
-<net name="DOUT" class="0">
-<segment>
-<pinref part="IC1" gate="G$1" pin="DOUT"/>
-<wire x1="45.72" y1="43.18" x2="38.1" y2="43.18" width="0.1524" layer="91"/>
-<label x="38.1" y="43.18" size="1.016" layer="95" ratio="0" rot="R180" xref="yes"/>
-</segment>
-</net>
 <net name="DIN" class="0">
 <segment>
@@
 <segment>
 <pinref part="VR1" gate="R?" pin="CW"/>
-<wire x1="38.1" y1="33.02" x2="38.1" y2="30.48" width="0.1524" layer="91"/>
+<wire x1="38.1" y1="33.02" x2="40.64" y2="33.02" width="0.1524" layer="91"/>
 <pinref part="GND2" gate="1" pin="GND"/>
 </segment>
@@
 <label x="50.8" y="78.74" size="1.016" layer="95" ratio="0" rot="R180" xref="yes"/>
 </segment>
-</net>
-<net name="D6" class="0">
-<segment>
-<pinref part="IC1" gate="G$1" pin="DIG5"/>
-<wire x1="73.66" y1="43.18" x2="81.28" y2="43.18" width="0.1524" layer="91"/>
-<label x="81.28" y="43.18" size="1.016" layer="95" ratio="0" xref="yes"/>
-<label x="81.28" y="43.18" size="1.016" layer="95" ratio="0" xref="yes"/>
+<segment>
+<pinref part="C1" gate="G$1" pin="2"/>
+<wire x1="-7.62" y1="25.4" x2="-7.62" y2="22.86" width="0.1524" layer="91"/>
+<label x="-7.62" y="22.86" size="1.016" layer="95" rot="R270" xref="yes"/>
 </segment>
 </net>
@@
 <label x="22.86" y="35.56" size="1.016" layer="95" rot="R90" xref="yes"/>
 </segment>
+<segment>
+<pinref part="C1" gate="G$1" pin="1"/>
+<wire x1="-7.62" y1="33.02" x2="-7.62" y2="35.56" width="0.1524" layer="91"/>
+<label x="-7.62" y="35.56" size="1.016" layer="95" rot="R90" xref="yes"/>
+</segment>
 </net>
 </nets>
 </sheet>
 </sheets>
+<errors>
+</errors>
 </schematic>
 </drawing>
